Commit message: Updated imav_env

File: imav_env/models/icarus.xacro (robot description, xacro)
@@ -21,5 +21,5 @@
   <xacro:property name="rotor_velocity_slowdown_sim" value="10" />
   <xacro:property name="use_mesh_file" value="true" />
-  <xacro:property name="mesh_file" value="package://imav_sim/meshes/firefly.dae" />
+  <xacro:property name="mesh_file" value="package://imav_env/meshes/firefly.dae" />
   <xacro:property name="mass" value="1.5" /> <!-- [kg] -->
   <xacro:property name="body_width" value="0.1" /> <!-- [m] -->
@@ -76,5 +76,5 @@
     rotor_drag_coefficient="${rotor_drag_coefficient}"
     rolling_moment_coefficient="${rolling_moment_coefficient}"
-    color="Yellow"
+    color="Red"
     use_own_mesh="false"
     mesh="">
@@ -179,5 +179,5 @@
     rotor_drag_coefficient="${rotor_drag_coefficient}"
     rolling_moment_coefficient="${rolling_moment_coefficient}"
-    color="Yellow"
+    color="Red"
     use_own_mesh="false"
     mesh="">

File: imav_env/models/icarus_base.xacro (robot description, xacro)
@@ -17,7 +17,7 @@
 -->
 <robot name="firefly" xmlns:xacro="http://ros.org/wiki/xacro">
-  <xacro:include filename="$(find imav_sim)/models/component_snippets.xacro" />
+  <xacro:include filename="$(find imav_env)/models/component_snippets.xacro" />
   <!-- Instantiate firefly "mechanics" -->
-  <xacro:include filename="$(find imav_sim)/models/icarus.xacro" />
+  <xacro:include filename="$(find imav_env)/models/icarus.xacro" />
   <!-- Instantiate a controller. -->
   <xacro:controller_plugin_macro namespace="${namespace}" imu_sub_topic="imu" />

File: imav_env/models/magnus.xacro (robot description, xacro)
@@ -21,5 +21,5 @@
   <xacro:property name="rotor_velocity_slowdown_sim" value="10" />
   <xacro:property name="use_mesh_file" value="true" />
-  <xacro:property name="mesh_file" value="package://imav_sim/meshes/firefly.dae" />
+  <xacro:property name="mesh_file" value="package://imav_env/meshes/firefly.dae" />
   <xacro:property name="mass" value="1.5" /> <!-- [kg] -->
   <xacro:property name="body_width" value="0.1" /> <!-- [m] -->
@@ -76,5 +76,5 @@
     rotor_drag_coefficient="${rotor_drag_coefficient}"
     rolling_moment_coefficient="${rolling_moment_coefficient}"
-    color="Red"
+    color="Yellow"
     use_own_mesh="false"
     mesh="">
@@ -179,5 +179,5 @@
     rotor_drag_coefficient="${rotor_drag_coefficient}"
     rolling_moment_coefficient="${rolling_moment_coefficient}"
-    color="Red"
+    color="Yellow"
     use_own_mesh="false"
     mesh="">

File: imav_env/models/magnus_base.xacro (robot description, xacro)
@@ -17,7 +17,7 @@
 -->
 <robot name="firefly" xmlns:xacro="http://ros.org/wiki/xacro">
-  <xacro:include filename="$(find imav_sim)/models/component_snippets.xacro" />
+  <xacro:include filename="$(find imav_env)/models/component_snippets.xacro" />
   <!-- Instantiate firefly "mechanics" -->
-  <xacro:include filename="$(find imav_sim)/models/vega.xacro" />
+  <xacro:include filename="$(find imav_env)/models/magnus.xacro" />
   <!-- Instantiate a controller. -->
   <xacro:controller_plugin_macro namespace="${namespace}" imu_sub_topic="imu" />

File: imav_env/models/multirotor_base.xacro (robot description, xacro)
@@ -97,5 +97,5 @@
           </xacro:if>
           <xacro:unless value="${use_own_mesh}">
-            <mesh filename="package://imav_sim/meshes/propeller_${direction}.dae"
+            <mesh filename="package://imav_env/meshes/propeller_${direction}.dae"
               scale="${radius_rotor} ${radius_rotor} ${radius_rotor}" /> <!-- The propeller meshes have a radius of 1m -->
             <!-- <box size="${2*radius_rotor} 0.01 0.005"/> -->

File: imav_env/models/vega.xacro (robot description, xacro)
@@ -21,5 +21,5 @@
   <xacro:property name="rotor_velocity_slowdown_sim" value="10" />
   <xacro:property name="use_mesh_file" value="true" />
-  <xacro:property name="mesh_file" value="package://imav_sim/meshes/firefly.dae" />
+  <xacro:property name="mesh_file" value="package://imav_env/meshes/firefly.dae" />
   <xacro:property name="mass" value="1.5" /> <!-- [kg] -->
   <xacro:property name="body_width" value="0.1" /> <!-- [m] -->

File: imav_env/models/vega_base.xacro (robot description, xacro)
@@ -17,7 +17,7 @@
 -->
 <robot name="firefly" xmlns:xacro="http://ros.org/wiki/xacro">
-  <xacro:include filename="$(find imav_sim)/models/component_snippets.xacro" />
+  <xacro:include filename="$(find imav_env)/models/component_snippets.xacro" />
   <!-- Instantiate firefly "mechanics" -->
-  <xacro:include filename="$(find imav_sim)/models/magnus.xacro" />
+  <xacro:include filename="$(find imav_env)/models/vega.xacro" />
   <!-- Instantiate a controller. -->
   <xacro:controller_plugin_macro namespace="${namespace}" imu_sub_topic="imu" />
